File: Eagle/PPMCapture.sch (EAGLE design)
At the start: 4 parts, among them U1 ATTINY85V-10P

Commit message: Chaned .1 header to JST 3pin connector
Parts:
- removed JP1, JP2, JP3: (no value), GTOR - Connectors:PINHD-1X3
- added U$1, U$2, U$3: JST-PH_3-PIN_HEADER, SRG:JST-PH_3-PIN_HEADER
Connections:
- net +5V: now also U$1.1, U$2.1, U$3.1; no longer JP1.1, JP2.1, JP3.1
- net GND: now also U$1.3, U$2.3, U$3.3; no longer JP1.3, JP2.3, JP3.3
- net LEDOUT: now also U$3.2; no longer JP3.2
- net PPM: now also U$1.2, U$2.2; no longer JP1.2, JP2.2
